File: PCB/01.30/RaspberryPi_Hat/RaspberryPi_Hat.kicad_sch (KiCad schematic)
At the start: 11 parts, among them J1 GPIO, J2 Conn_01x03, J3 Conn_01x02, J4 Conn_01x02, J5 Conn_01x05, J6 Conn_01x03, U1 CAT24C256

Commit message: Finished PCB implementation
Connections:
- net S0 is gone; now on net GPIO17: J5.3 (Pin_3)
- net S1 is gone; now on net GPIO27: J5.2 (Pin_2)
Other:
- note added: "Battery"
- note added: "Greyscale Sensor"
- note added: "Interruptor"
- note added: "Motor"
Changed lines of the file:
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@@
 		(date "15 nov 2012")
+	)
+	(text "Battery"
+		(exclude_from_sim no)
+		(at 136.398 73.914 0)
+		(effects
+			(font
+				(size 1.27 1.27)
+			)
+		)
+	)
+	(text "Greyscale Sensor\n"
+		(exclude_from_sim no)
+		(at 139.954 112.014 0)
+		(effects
+			(font
+				(size 1.27 1.27)
+			)
+		)
 	)
 	(text "Additional pin functions:\nhttps://pinout.xyz/"
@@
 		)
 	)
+	(text "Motor"
+		(exclude_from_sim no)
+		(at 134.112 86.106 0)
+		(effects
+			(font
+				(size 1.27 1.27)
+			)
+		)
+	)
 	(text "ID_SD and ID_SC PINS:\nThese pins are reserved for HAT ID EEPROM.\n\nAt boot time this I2C interface will be\ninterrogated to look for an EEPROM\nthat identifes the attached board and\nallows automagic setup of the GPIOs\n(and optionally, Linux drivers).\n\nBridging JP1 enables write protection.\n\nDO NOT USE these pins for anything other\nthan attaching an I2C ID EEPROM. Leave\nunconnected if ID EEPROM not required."
 		(exclude_from_sim no)
@@
 		)
 	)
+	(text "Interruptor"
+		(exclude_from_sim no)
+		(at 134.366 102.362 0)
+		(effects
+			(font
+				(size 1.27 1.27)
+			)
+		)
+	)
 	(text "S0 → GPIO17\nS1 → GPIO27\nS2 → GPIO22\nVCC → +3V3 (Can be wired to either Pin 1 or 17)\nGND → GND ( Can be wired to either Pin 9,25,39,6,14,20,30,34)"
 		(exclude_from_sim no)
@@
 	)
 	(junction
+		(at 76.2 80.01)
+		(diameter 0)
+		(color 0 0 0 0)
+	)
+	(junction
 		(at 120.65 115.57)
 		(diameter 0)
@@
 	)
 	(junction
+		(at 48.26 27.94)
+		(diameter 0)
+		(color 0 0 0 0)
+	)
+	(junction
 		(at 93.98 165.1)
 		(diameter 1.016)
@@
 	(wire
 		(pts
+			(xy 26.67 96.52) (xy 26.67 43.18)
+		)
+		(stroke
+			(width 0)
+			(type default)
+		)
+	)
+	(wire
+		(pts
+			(xy 48.26 27.94) (xy 55.88 27.94)
+		)
+		(stroke
+			(width 0)
+			(type default)
+		)
+	)
+	(wire
+		(pts
 			(xy 76.2 63.5) (xy 76.2 68.58)
 		)
@@
 	(wire
 		(pts
+			(xy 26.67 96.52) (xy 121.92 96.52)
+		)
+		(stroke
+			(width 0)
+			(type default)
+		)
+	)
+	(wire
+		(pts
+			(xy 121.92 101.6) (xy 106.68 101.6)
+		)
+		(stroke
+			(width 0)
+			(type default)
+		)
+	)
+	(wire
+		(pts
 			(xy 60.96 60.96) (xy 31.75 60.96)
 		)
@@
 	(wire
 		(pts
+			(xy 81.28 104.14) (xy 81.28 80.01)
+		)
+		(stroke
+			(width 0)
+			(type default)
+		)
+	)
+	(wire
+		(pts
 			(xy 58.42 58.42) (xy 60.96 58.42)
 		)
@@
 	(wire
 		(pts
+			(xy 27.94 93.98) (xy 27.94 45.72)
+		)
+		(stroke
+			(width 0)
+			(type default)
+		)
+	)
+	(wire
+		(pts
 			(xy 120.65 113.03) (xy 121.92 113.03)
 		)
@@
 	(wire
 		(pts
+			(xy 121.92 99.06) (xy 25.4 99.06)
+		)
+		(stroke
+			(width 0)
+			(type default)
+		)
+	)
+	(wire
+		(pts
 			(xy 73.66 45.72) (xy 100.33 45.72)
 		)
@@
 	(wire
 		(pts
+			(xy 48.26 17.78) (xy 106.68 17.78)
+		)
+		(stroke
+			(width 0)
+			(type default)
+		)
+	)
+	(wire
+		(pts
 			(xy 73.66 76.2) (xy 100.33 76.2)
 		)
@@
 	(wire
 		(pts
-			(xy 31.75 43.18) (xy 60.96 43.18)
-		)
-		(stroke
-			(width 0)
-			(type solid)
-		)
-	)
-	(wire
-		(pts
 			(xy 101.6 172.72) (xy 101.6 177.8)
 		)
@@
 	(wire
 		(pts
+			(xy 81.28 80.01) (xy 76.2 80.01)
+		)
+		(stroke
+			(width 0)
+			(type default)
+		)
+	)
+	(wire
+		(pts
 			(xy 20.32 115.57) (xy 20.32 63.5)
 		)
@@
 	(wire
 		(pts
-			(xy 16.51 27.94) (xy 55.88 27.94)
+			(xy 16.51 27.94) (xy 48.26 27.94)
 		)
 		(stroke
@@
 	(wire
 		(pts
+			(xy 25.4 99.06) (xy 25.4 40.64)
+		)
+		(stroke
+			(width 0)
+			(type default)
+		)
+	)
+	(wire
+		(pts
 			(xy 76.2 27.94) (xy 76.2 30.48)
 		)
@@
 	(wire
 		(pts
+			(xy 27.94 45.72) (xy 60.96 45.72)
+		)
+		(stroke
+			(width 0)
+			(type default)
+		)
+	)
+	(wire
+		(pts
 			(xy 76.2 24.13) (xy 76.2 27.94)
 		)
@@
 	(wire
 		(pts
-			(xy 31.75 45.72) (xy 60.96 45.72)
-		)
-		(stroke
-			(width 0)
-			(type solid)
-		)
-	)
-	(wire
-		(pts
 			(xy 49.53 113.03) (xy 120.65 113.03)
 		)
@@
 	(wire
 		(pts
+			(xy 106.68 101.6) (xy 106.68 17.78)
+		)
+		(stroke
+			(width 0)
+			(type default)
+		)
+	)
+	(wire
+		(pts
 			(xy 31.75 66.04) (xy 60.96 66.04)
 		)
@@
 	(wire
 		(pts
+			(xy 48.26 17.78) (xy 48.26 27.94)
+		)
+		(stroke
+			(width 0)
+			(type default)
+		)
+	)
+	(wire
+		(pts
 			(xy 76.2 30.48) (xy 73.66 30.48)
 		)
@@
 	(wire
 		(pts
+			(xy 110.49 93.98) (xy 27.94 93.98)
+		)
+		(stroke
+			(width 0)
+			(type default)
+		)
+	)
+	(wire
+		(pts
 			(xy 81.28 185.42) (xy 81.28 187.96)
 		)
@@
 	(wire
 		(pts
+			(xy 26.67 43.18) (xy 60.96 43.18)
+		)
+		(stroke
+			(width 0)
+			(type default)
+		)
+	)
+	(wire
+		(pts
 			(xy 55.88 27.94) (xy 60.96 27.94)
 		)
@@
 		)
 	)
+	(wire
+		(pts
+			(xy 121.92 104.14) (xy 81.28 104.14)
+		)
+		(stroke
+			(width 0)
+			(type default)
+		)
+	)

Commit message: added minor tweak to pcb
Connections:
- net S2 is gone; now on net GPIO22: J5.1 (Pin_1)
- no-connect marks 3 -> 5
Changed lines of the file:
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@@
 		(at 71.12 180.34)
 	)
+	(no_connect
+		(at 86.36 114.3)
+	)
+	(no_connect
+		(at 86.36 102.87)
+	)
 	(wire
 		(pts
@@
 	(wire
 		(pts
-			(xy 110.49 93.98) (xy 27.94 93.98)
-		)
-		(stroke
+			(xy 27.94 93.98) (xy 121.92 93.98)
+		)
+		(stroke
