File: PCB/01.30/RaspberryPi_Hat/RaspberryPi_Hat.kicad_pcb (KiCad board)
At the start: 2 copper layers, 65 x 56 mm, 10 parts, among them J1 GPIO, J2 Conn_01x03, J3 Conn_01x02, J4 Conn_01x02, J5 Conn_01x05, J6 Conn_01x03

Commit message: PCB Layout updated
Parts:
- moved J2 25.2 mm to (112.5, 75.0)
- moved J4 22.8 mm to (130.5, 75.5)
- moved J6 15.5 mm to (134.0, 60.5), turned to 90 degrees
- moved J3 5.81 mm to (122.0, 76.0)
Routing:
- net GND: track 9.78 -> 65.3 mm
- net +3V3: track 22.0 -> 39.0 mm
- net /GPIO5: track 0.00 -> 16.1 mm
Changed lines of the file:
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@@
 	(footprint "Connector_PinHeader_2.54mm:PinHeader_1x03_P2.54mm_Vertical"
 		(layer "F.Cu")
-		(at 137 69)
+		(at 112.5 74.96)
 		(descr "Through hole straight pin header, 1x03, 2.54mm pitch, single row")
 		(tags "Through hole pin header THT 1x03 2.54mm single row")
@@
 	(footprint "Connector_PinHeader_2.54mm:PinHeader_1x03_P2.54mm_Vertical"
 		(layer "F.Cu")
-		(at 147 68.92)
+		(at 133.96 60.5 90)
 		(descr "Through hole straight pin header, 1x03, 2.54mm pitch, single row")
 		(tags "Through hole pin header THT 1x03 2.54mm single row")
 		(property "Reference" "J6"
-			(at 0 -2.38 0)
+			(at 0 -2.38 90)
 			(layer "F.SilkS")
 			(effects
@@
 		)
 		(property "Value" "Conn_01x03"
-			(at 0 7.46 0)
+			(at 0 7.46 90)
 			(layer "F.Fab")
 			(effects
@@
 		)
 		(property "Datasheet" "~"
-			(at 0 0 0)
+			(at 0 0 90)
 			(layer "F.Fab")
 			(hide yes)
@@
 		)
 		(property "Description" "Generic connector, single row, 01x03, script generated (kicad-library-utils/schlib/autogen/connector/)"
-			(at 0 0 0)
+			(at 0 0 90)
 			(layer "F.Fab")
 			(hide yes)
@@
 		)
 		(fp_line
+			(start 1.38 1.27)
+			(end 1.38 6.46)
+			(stroke
+				(width 0.12)
+				(type solid)
+			)
+			(layer "F.SilkS")
+		)
+		(fp_line
+			(start -1.38 1.27)
+			(end 1.38 1.27)
+			(stroke
+				(width 0.12)
+				(type solid)
+			)
+			(layer "F.SilkS")
+		)
+		(fp_line
 			(start -1.38 1.27)
 			(end -1.38 6.46)
@@
 		)
 		(fp_line
-			(start -1.38 1.27)
-			(end 1.38 1.27)
-			(stroke
-				(width 0.12)
-				(type solid)
-			)
-			(layer "F.SilkS")
-		)
-		(fp_line
 			(start -1.38 6.46)
-			(end 1.38 6.46)
-			(stroke
-				(width 0.12)
-				(type solid)
-			)
-			(layer "F.SilkS")
-		)
-		(fp_line
-			(start 1.38 1.27)
 			(end 1.38 6.46)
 			(stroke
@@
 		)
 		(fp_line
+			(start 1.27 -1.27)
+			(end 1.27 6.35)
+			(stroke
+				(width 0.1)
+				(type solid)
+			)
+			(layer "F.Fab")
+		)
+		(fp_line
+			(start -0.635 -1.27)
+			(end 1.27 -1.27)
+			(stroke
+				(width 0.1)
+				(type solid)
+			)
+			(layer "F.Fab")
+		)
+		(fp_line
 			(start -1.27 -0.635)
 			(end -0.635 -1.27)
@@
 		)
 		(fp_line
+			(start 1.27 6.35)
+			(end -1.27 6.35)
+			(stroke
+				(width 0.1)
+				(type solid)
+			)
+			(layer "F.Fab")
+		)
+		(fp_line
 			(start -1.27 6.35)
 			(end -1.27 -0.635)
@@
 			(layer "F.Fab")
 		)
-		(fp_line
-			(start -0.635 -1.27)
-			(end 1.27 -1.27)
-			(stroke
-				(width 0.1)
-				(type solid)
-			)
-			(layer "F.Fab")
-		)
-		(fp_line
-			(start 1.27 -1.27)
-			(end 1.27 6.35)
-			(stroke
-				(width 0.1)
-				(type solid)
-			)
-			(layer "F.Fab")
-		)
-		(fp_line
-			(start 1.27 6.35)
-			(end -1.27 6.35)
-			(stroke
-				(width 0.1)
-				(type solid)
-			)
-			(layer "F.Fab")
-		)
 		(fp_text user "${REFERENCE}"
-			(at 0 2.54 90)
+			(at 0 2.54 0)
 			(layer "F.Fab")
 			(effects
@@
 		)
 		(pad "1" thru_hole rect
-			(at 0 0)
+			(at 0 0 90)
 			(size 1.7 1.7)
 			(drill 1)
@@
 		)
 		(pad "2" thru_hole circle
-			(at 0 2.54)
+			(at 0 2.54 90)
 			(size 1.7 1.7)
 			(drill 1)
@@
 		)
 		(pad "3" thru_hole circle
-			(at 0 5.08)
+			(at 0 5.08 90)
 			(size 1.7 1.7)
 			(drill 1)
@@
 	(footprint "Connector_PinHeader_2.54mm:PinHeader_1x02_P2.54mm_Vertical"
 		(layer "F.Cu")
-		(at 141.5 55.46)
+		(at 130.5 75.46)
 		(descr "Through hole straight pin header, 1x02, 2.54mm pitch, single row")
 		(tags "Through hole pin header THT 1x02 2.54mm single row")
@@
 	(footprint "Connector_PinHeader_2.54mm:PinHeader_1x02_P2.54mm_Vertical"
 		(layer "F.Cu")
-		(at 124 70.5)
+		(at 122 75.96)
 		(descr "Through hole straight pin header, 1x02, 2.54mm pitch, single row")
 		(tags "Through hole pin header THT 1x02 2.54mm single row")
@@
 	)
 	(segment
+		(start 156.563251 72.499642)
+		(end 156.609121 72.453772)
+		(width 0.2)
+		(layer "F.Cu")
+		(net 1)
+	)
+	(segment
+		(start 136.5 60.77)
+		(end 136.5 72.5)
+		(width 0.2)
+		(layer "F.Cu")
+		(net 1)
+	)
+	(segment
+		(start 156.63 48.77)
+		(end 156.63 72.432892)
+		(width 0.2)
+		(layer "F.Cu")
+		(net 1)
+	)
+	(segment
 		(start 115.92 51.58)
 		(end 116 51.5)
@@
 	)
 	(segment
+		(start 156.63 72.432892)
+		(end 156.596446 72.466446)
+		(width 0.2)
+		(layer "F.Cu")
+		(net 1)
+	)
+	(segment
+		(start 136.576666 72.499642)
+		(end 156.563251 72.499642)
+		(width 0.2)
+		(layer "F.Cu")
+		(net 1)
+	)
+	(segment
 		(start 116 51.5)
 		(end 118.5 51.5)
@@
 		(layer "F.Cu")
 		(net 1)
+	)
+	(segment
+		(start 143.93 54.5005)
+		(end 143.93 48.77)
+		(width 0.2)
+		(layer "F.Cu")
+		(net 21)
+	)
+	(segment
+		(start 144.4995 49.24975)
+		(end 144 48.75025)
+		(width 0.2)
+		(layer "F.Cu")
+		(net 21)
+	)
+	(segment
+		(start 143.73 48.77)
+		(end 143.93 48.77)
+		(width 0.2)
+		(layer "F.Cu")
+		(net 21)
+	)
+	(segment
+		(start 139 59)
+		(end 139 54.5005)
+		(width 0.2)
+		(layer "F.Cu")
+		(net 21)
+	)
+	(segment
+		(start 139 54.5005)
+		(end 143.93 54.5005)
+		(width 0.2)
+		(layer "F.Cu")
+		(net 21)
 	)
 	(segment
@@
 		(width 0.2)
 		(layer "F.Cu")
+		(net 31)
+	)
+	(segment
+		(start 128.69 48.77)
+		(end 128.69 60.5)
+		(width 0.2)
+		(layer "F.Cu")
+		(net 31)
+	)
+	(segment
+		(start 128.69 60.5)
+		(end 133.965 60.5)
+		(width 0.2)
+		(layer "F.Cu")
